Commit message: added transformation to staplerspitze

File: src/SC-LIO-SAM/SC-LIO-SAM/launch/include/config/robot.urdf.xacro (robot description, xacro)
@@ -27,3 +27,15 @@
     <origin xyz="0 0 0" rpy="0 0 0" />
   </joint>
+  <link name="lidar_link"> </link>
+  <joint name="lidar_joint" type="fixed">
+    <parent link="chassis_link" />
+    <child link="lidar_link" />
+    <origin xyz="0 0 0" rpy="0 0 0" />
+  </joint>
+  <link name="spitze_link"> </link>
+  <joint name="spitze_joint" type="fixed">
+    <parent link="chassis_link" />
+    <child link="spitze_link" />
+    <origin xyz="0 0 0" rpy="0 0 0" />
+  </joint>
 </robot>

Commit message: Added transformation to axis for testing

File: src/SC-LIO-SAM/SC-LIO-SAM/launch/include/config/robot.urdf.xacro (robot description, xacro)
@@ -33,8 +33,8 @@
     <origin xyz="0 0 0" rpy="0 0 0" />
   </joint>
-  <link name="spitze_link"> </link>
-  <joint name="spitze_joint" type="fixed">
+  <link name="axis_link"> </link>
+  <joint name="axis_joint" type="fixed">
     <parent link="chassis_link" />
-    <child link="spitze_link" />
+    <child link="axis_link" />
     <origin xyz="0 0 0" rpy="0 0 0" />
   </joint>
